File: Schematics/BSPD.kicad_sch (KiCad schematic)
At the start: 0 parts

Commit message: UPDATE
Parts:
- added C? (x4): 100nF, Capacitor_THT:CP_Axial_L10.0mm_D4.5mm_P15.00mm_Horizontal, symbol Device:C_Small
- added C?: CP, symbol Device:CP
- added C?: 330uF, Capacitor_THT:CP_Axial_L10.0mm_D4.5mm_P15.00mm_Horizontal, symbol Device:C_Small
- added R?: R, symbol Device:R
- added R?: 1K, Resistor_THT:R_Axial_DIN0204_L3.6mm_D1.6mm_P5.08mm_Horizontal, symbol Device:R_US
- added R? (x2): 1k, Resistor_THT:R_Axial_DIN0204_L3.6mm_D1.6mm_P5.08mm_Horizontal, symbol Device:R_US
- added R?: 2k2, Resistor_THT:R_Axial_DIN0204_L3.6mm_D1.6mm_P5.08mm_Horizontal, symbol Device:R_US
- added U? (x3): 74LVC1G08, symbol 74xGxx:74LVC1G08
- added U?: LMV7219M5, Package_TO_SOT_SMD:SOT-23-5, symbol Comparator:LMV7219M5
- added U?: NE555D, Package_SO:SOIC-8_3.9x4.9mm_P1.27mm, symbol Timer:NE555D
Connections:
- net BSPD_FAULT: now also U?.4, U?.7 (DIS)
- new net: R?.2, U?.1, U?.4
- new net: C?.1, U?.4, U?.4 (R), U?.8 (VCC)
- new net: C?.2, R?.2, U?.2 (TR), U?.6 (THR)
- new net: R?.1, U?.1, U?.2
- new net: C?.1, R?.1, U?.3 (+)
- new net: R?.1, R?.2, U?.4 (-)
- new net +5V: C?.2, C?.2, C?.2, C?.2, R?.2, R?.2, U?.5 (V+), U?.5 (VCC), U?.5 (VCC), U?.5 (VCC)
- new net Earth: C?.1, C?.1, C?.1, C?.1, C?.2, R?.1, R?.1, U?.1 (GND), U?.2 (V-), U?.3 (GND), U?.3 (GND), U?.3 (GND)
- new net HALL: U?.1, U?.1
- new net Sheet61EFC276/Brake_Signal: U?.2
- new net Sheet61EFC277/Brake_Sensor_Output: U?.2
Other:
- added sheet Sheet61EFC276 (bspd_brake sense.kicad_sch)
- added sheet Sheet61EFC277 (bspd_brake sense.kicad_sch)
