File: Schematics/DASHBOARD.kicad_sch (KiCad schematic)
At the start: 0 parts

Commit message: REFACTOR
Parts:
- added RESET2: SW_DPST_x2, symbol Switch:SW_Push
- added U7: STM32F407VETx, Package_QFP:LQFP-100_14x14mm_P0.5mm, symbol MCU_ST_STM32F4:STM32F407VETx
Connections:
- new net GND: RESET2.1
- new net SHUTDOWN_RESET: RESET2.2
Changed lines of the file:
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@@
 (kicad_sch (version 20211123) (generator eeschema)
   (paper "A4")
+  (wire (pts (xy 142.24 110.49) (xy 146.05 110.49))
+    (stroke (width 0) (type default) (color 0 0 0 0))
+  )
+  (wire (pts (xy 129.54 110.49) (xy 132.08 110.49))
+    (stroke (width 0) (type default) (color 0 0 0 0))
+  )
+  (hierarchical_label "BMS_LED" (shape input) (at 132.08 74.93 0)
+    (effects (font (size 1.27 1.27) (thickness 0.254) bold) (justify left))
+  )
+  (hierarchical_label "SIG_RPS" (shape input) (at 179.07 78.74 0)
+    (effects (font (size 1.27 1.27) (thickness 0.254) bold) (justify left))
+  )
+  (hierarchical_label "GND_RPS" (shape output) (at 179.07 81.28 0)
+    (effects (font (size 1.27 1.27) (thickness 0.254) bold) (justify left))
+  )
+  (hierarchical_label "SIG_APPS" (shape input) (at 179.07 68.58 0)
+    (effects (font (size 1.27 1.27) (thickness 0.254) bold) (justify left))
+  )
+  (hierarchical_label "GND" (shape input) (at 132.08 57.15 0)
+    (effects (font (size 1.27 1.27) (thickness 0.254) bold) (justify left))
+  )
+  (hierarchical_label "LV_ACTIVE" (shape input) (at 132.08 62.23 0)
+    (effects (font (size 1.27 1.27) (thickness 0.254) bold) (justify left))
+  )
+  (hierarchical_label "5V_APPS" (shape output) (at 179.07 66.04 0)
+    (effects (font (size 1.27 1.27) (thickness 0.254) bold) (justify left))
+  )
+  (hierarchical_label "BRAKE" (shape input) (at 179.07 60.96 0)
+    (effects (font (size 1.27 1.27) (thickness 0.254) bold) (justify left))
+  )
+  (hierarchical_label "LV" (shape input) (at 132.08 59.69 0)
+    (effects (font (size 1.27 1.27) (thickness 0.254) bold) (justify left))
+  )
+  (hierarchical_label "ACC" (shape output) (at 179.07 58.42 0)
+    (effects (font (size 1.27 1.27) (thickness 0.254) bold) (justify left))
+  )
+  (hierarchical_label "HVD_LED" (shape input) (at 132.08 82.55 0)
+    (effects (font (size 1.27 1.27) (thickness 0.254) bold) (justify left))
+  )
+  (hierarchical_label "5V_RPS" (shape output) (at 179.07 76.2 0)
+    (effects (font (size 1.27 1.27) (thickness 0.254) bold) (justify left))
+  )
+  (hierarchical_label "IMD_LED" (shape input) (at 132.08 71.12 0)
+    (effects (font (size 1.27 1.27) (thickness 0.254) bold) (justify left))
+  )
+  (hierarchical_label "CRITICAL_LED" (shape input) (at 132.08 67.31 0)
+    (effects (font (size 1.27 1.27) (thickness 0.254) bold) (justify left))
+  )
+  (hierarchical_label "BSPD_LED" (shape input) (at 132.08 78.74 0)
+    (effects (font (size 1.27 1.27) (thickness 0.254) bold) (justify left))
+  )
+  (hierarchical_label "GND_APPS" (shape output) (at 179.07 71.12 0)
+    (effects (font (size 1.27 1.27) (thickness 0.254) bold) (justify left))
+  )
+  (hierarchical_label "ＣＡＮ＿Ｈ" (shape input) (at 132.08 87.63 0)
+    (effects (font (size 1.27 1.27) (thickness 0.254) bold) (justify left))
+  )
+  (hierarchical_label "ＣＡＮ＿Ｌ" (shape input) (at 132.08 90.17 0)
+    (effects (font (size 1.27 1.27) (thickness 0.254) bold) (justify left))
+  )
+  (hierarchical_label "SHUTDOWN_RESET" (shape output) (at 146.05 110.49 0)
+    (effects (font (size 1.27 1.27) (thickness 0.254) bold) (justify left))
+  )
+  (symbol (lib_id "power:GND") (at 129.54 110.49 0)
+    (in_bom yes) (on_board yes)
+    (property "Reference" "#PWR08" (id 0) (at 129.54 116.84 0)
+      (effects (font (size 1.27 1.27)) hide)
+    )
+    (property "Value" "GND" (id 1) (at 129.54 114.3 0))
+    (property "Footprint" "" (id 2) (at 129.54 110.49 0)
+      (effects (font (size 1.27 1.27)) hide)
+    )
+    (property "Datasheet" "" (id 3) (at 129.54 110.49 0)
+      (effects (font (size 1.27 1.27)) hide)
+    )
+    (pin "1")
+  )
+  (symbol (lib_id "MCU_ST_STM32F4:STM32F407VETx") (at 77.47 104.14 0)
+    (in_bom yes) (on_board yes) (fields_autoplaced)
+    (property "Reference" "U7" (id 0) (at 84.5694 172.3295 0)
+      (effects (font (size 1.27 1.27)) (justify left))
+    )
+    (property "Value" "STM32F407VETx" (id 1) (at 84.5694 175.1046 0)
+      (effects (font (size 1.27 1.27)) (justify left))
+    )
+    (property "Footprint" "Package_QFP:LQFP-100_14x14mm_P0.5mm" (id 2) (at 59.69 170.18 0)
+      (effects (font (size 1.27 1.27)) (justify right) hide)
+    )
+    (property "Datasheet" "http://www.st.com/st-web-ui/static/active/en/resource/technical/document/datasheet/DM00037051.pdf" (id 3) (at 77.47 104.14 0)
+      (effects (font (size 1.27 1.27)) hide)
+    )
+    (pin "1")
+    (pin "10")
+    (pin "100")
+    (pin "11")
+    (pin "12")
+    (pin "13")
+    (pin "14")
+    (pin "15")
+    (pin "16")
+    (pin "17")
+    (pin "18")
+    (pin "19")
+    (pin "2")
+    (pin "20")
+    (pin "21")
+    (pin "22")
+    (pin "23")
+    (pin "24")
+    (pin "25")
+    (pin "26")
+    (pin "27")
+    (pin "28")
+    (pin "29")
+    (pin "3")
+    (pin "30")
+    (pin "31")
+    (pin "32")
+    (pin "33")
+    (pin "34")
+    (pin "35")
+    (pin "36")
+    (pin "37")
+    (pin "38")
+    (pin "39")
+    (pin "4")
+    (pin "40")
+    (pin "41")
+    (pin "42")
+    (pin "43")
+    (pin "44")
+    (pin "45")
+    (pin "46")
+    (pin "47")
+    (pin "48")
+    (pin "49")
+    (pin "5")
+    (pin "50")
+    (pin "51")
+    (pin "52")
+    (pin "53")
+    (pin "54")
+    (pin "55")
+    (pin "56")
+    (pin "57")
+    (pin "58")
+    (pin "59")
+    (pin "6")
+    (pin "60")
+    (pin "61")
+    (pin "62")
+    (pin "63")
+    (pin "64")
+    (pin "65")
+    (pin "66")
+    (pin "67")
+    (pin "68")
+    (pin "69")
+    (pin "7")
+    (pin "70")
+    (pin "71")
+    (pin "72")
+    (pin "73")
+    (pin "74")
+    (pin "75")
+    (pin "76")
+    (pin "77")
+    (pin "78")
+    (pin "79")
+    (pin "8")
+    (pin "80")
+    (pin "81")
+    (pin "82")
+    (pin "83")
+    (pin "84")
+    (pin "85")
+    (pin "86")
+    (pin "87")
+    (pin "88")
+    (pin "89")
+    (pin "9")
+    (pin "90")
+    (pin "91")
+    (pin "92")
+    (pin "93")
+    (pin "94")
+    (pin "95")
+    (pin "96")
+    (pin "97")
+    (pin "98")
+    (pin "99")
+  )
+  (symbol (lib_id "Switch:SW_Push") (at 137.16 110.49 0)
+    (in_bom yes) (on_board yes)
+    (property "Reference" "RESET2" (id 0) (at 137.16 105.5878 0))
+    (property "Value" "SW_DPST_x2" (id 1) (at 137.16 106.8324 0)
+      (effects (font (size 1.27 1.27)) hide)
+    )
+    (property "Footprint" "" (id 2) (at 137.16 110.49 0)
+      (effects (font (size 1.27 1.27)) hide)
+    )
+    (property "Datasheet" "~" (id 3) (at 137.16 110.49 0)
+      (effects (font (size 1.27 1.27)) hide)
+    )
+    (pin "1")
+    (pin "2")
+  )
 )

Commit message: UPDATE
Parts:
- removed RESET2: SW_DPST_x2, symbol Switch:SW_Push
- added R?: R_US, symbol Device:R_US
Connections:
- net CRITICAL_LED: now also R?.2
Changed lines of the file:
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@@
 (kicad_sch (version 20211123) (generator eeschema)
   (paper "A4")
-  (wire (pts (xy 142.24 110.49) (xy 146.05 110.49))
+  (wire (pts (xy 179.07 64.77) (xy 181.61 64.77))
     (stroke (width 0) (type default) (color 0 0 0 0))
   )
-  (wire (pts (xy 129.54 110.49) (xy 132.08 110.49))
-    (stroke (width 0) (type default) (color 0 0 0 0))
+  (global_label "CRITICAL_LED" (shape output) (at 224.79 64.77 180) (fields_autoplaced)
+    (effects (font (size 1.27 1.27)) (justify right))
+    (property "Intersheet References" "${INTERSHEET_REFS}" (id 0) (at 209.8583 64.6906 0)
+      (effects (font (size 1.27 1.27)) (justify right) hide)
+    )
   )
-  (hierarchical_label "BMS_LED" (shape input) (at 132.08 74.93 0)
+  (global_label "CRITICAL_LED" (shape input) (at 181.61 64.77 0) (fields_autoplaced)
+    (effects (font (size 1.27 1.27)) (justify left))
+    (property "Intersheet References" "${INTERSHEET_REFS}" (id 0) (at 196.5417 64.6906 0)
+      (effects (font (size 1.27 1.27)) (justify left) hide)
+    )
+  )
+  (hierarchical_label "BMS_LED" (shape input) (at 224.79 72.39 0)
     (effects (font (size 1.27 1.27) (thickness 0.254) bold) (justify left))
   )
-  (hierarchical_label "SIG_RPS" (shape input) (at 179.07 78.74 0)
+  (hierarchical_label "GND" (shape input) (at 224.79 54.61 0)
     (effects (font (size 1.27 1.27) (thickness 0.254) bold) (justify left))
   )
-  (hierarchical_label "GND_RPS" (shape output) (at 179.07 81.28 0)
+  (hierarchical_label "LV_ACTIVE" (shape input) (at 224.79 59.69 0)
     (effects (font (size 1.27 1.27) (thickness 0.254) bold) (justify left))
   )
-  (hierarchical_label "SIG_APPS" (shape input) (at 179.07 68.58 0)
+  (hierarchical_label "LV" (shape input) (at 224.79 57.15 0)
     (effects (font (size 1.27 1.27) (thickness 0.254) bold) (justify left))
   )
-  (hierarchical_label "GND" (shape input) (at 132.08 57.15 0)
+  (hierarchical_label "HVD_LED" (shape input) (at 224.79 80.01 0)
     (effects (font (size 1.27 1.27) (thickness 0.254) bold) (justify left))
   )
-  (hierarchical_label "LV_ACTIVE" (shape input) (at 132.08 62.23 0)
+  (hierarchical_label "IMD_LED" (shape input) (at 224.79 68.58 0)
     (effects (font (size 1.27 1.27) (thickness 0.254) bold) (justify left))
   )
-  (hierarchical_label "5V_APPS" (shape output) (at 179.07 66.04 0)
+  (hierarchical_label "CRITICAL_LED" (shape input) (at 224.79 64.77 0)
     (effects (font (size 1.27 1.27) (thickness 0.254) bold) (justify left))
   )
-  (hierarchical_label "BRAKE" (shape input) (at 179.07 60.96 0)
+  (hierarchical_label "BSPD_LED" (shape input) (at 224.79 76.2 0)
     (effects (font (size 1.27 1.27) (thickness 0.254) bold) (justify left))
   )
-  (hierarchical_label "LV" (shape input) (at 132.08 59.69 0)
+  (hierarchical_label "ＣＡＮ＿Ｈ" (shape input) (at 224.79 85.09 0)
     (effects (font (size 1.27 1.27) (thickness 0.254) bold) (justify left))
   )
-  (hierarchical_label "ACC" (shape output) (at 179.07 58.42 0)
+  (hierarchical_label "ＣＡＮ＿Ｌ" (shape input) (at 224.79 87.63 0)
     (effects (font (size 1.27 1.27) (thickness 0.254) bold) (justify left))
   )
-  (hierarchical_label "HVD_LED" (shape input) (at 132.08 82.55 0)
-    (effects (font (size 1.27 1.27) (thickness 0.254) bold) (justify left))
-  )
-  (hierarchical_label "5V_RPS" (shape output) (at 179.07 76.2 0)
-    (effects (font (size 1.27 1.27) (thickness 0.254) bold) (justify left))
-  )
-  (hierarchical_label "IMD_LED" (shape input) (at 132.08 71.12 0)
-    (effects (font (size 1.27 1.27) (thickness 0.254) bold) (justify left))
-  )
-  (hierarchical_label "CRITICAL_LED" (shape input) (at 132.08 67.31 0)
-    (effects (font (size 1.27 1.27) (thickness 0.254) bold) (justify left))
-  )
-  (hierarchical_label "BSPD_LED" (shape input) (at 132.08 78.74 0)
-    (effects (font (size 1.27 1.27) (thickness 0.254) bold) (justify left))
-  )
-  (hierarchical_label "GND_APPS" (shape output) (at 179.07 71.12 0)
-    (effects (font (size 1.27 1.27) (thickness 0.254) bold) (justify left))
-  )
-  (hierarchical_label "ＣＡＮ＿Ｈ" (shape input) (at 132.08 87.63 0)
-    (effects (font (size 1.27 1.27) (thickness 0.254) bold) (justify left))
-  )
-  (hierarchical_label "ＣＡＮ＿Ｌ" (shape input) (at 132.08 90.17 0)
-    (effects (font (size 1.27 1.27) (thickness 0.254) bold) (justify left))
-  )
-  (hierarchical_label "SHUTDOWN_RESET" (shape output) (at 146.05 110.49 0)
-    (effects (font (size 1.27 1.27) (thickness 0.254) bold) (justify left))
-  )
-  (symbol (lib_id "power:GND") (at 129.54 110.49 0)
-    (in_bom yes) (on_board yes)
-    (property "Reference" "#PWR08" (id 0) (at 129.54 116.84 0)
-      (effects (font (size 1.27 1.27)) hide)
-    )
-    (property "Value" "GND" (id 1) (at 129.54 114.3 0))
-    (property "Footprint" "" (id 2) (at 129.54 110.49 0)
-      (effects (font (size 1.27 1.27)) hide)
-    )
-    (property "Datasheet" "" (id 3) (at 129.54 110.49 0)
-      (effects (font (size 1.27 1.27)) hide)
-    )
-    (pin "1")
-  )
-  (symbol (lib_id "MCU_ST_STM32F4:STM32F407VETx") (at 77.47 104.14 0)
+  (symbol (lib_id "MCU_ST_STM32F4:STM32F407VETx") (at 77.47 104.14 0) (unit 1)
     (in_bom yes) (on_board yes) (fields_autoplaced)
     (property "Reference" "U7" (id 0) (at 84.5694 172.3295 0)
@@
     (pin "99")
   )
-  (symbol (lib_id "Switch:SW_Push") (at 137.16 110.49 0)
-    (in_bom yes) (on_board yes)
-    (property "Reference" "RESET2" (id 0) (at 137.16 105.5878 0))
-    (property "Value" "SW_DPST_x2" (id 1) (at 137.16 106.8324 0)
+  (symbol (lib_id "Device:R_US") (at 175.26 64.77 90) (mirror x) (unit 1)
+    (in_bom yes) (on_board yes) (fields_autoplaced)
+    (property "Reference" "R?" (id 0) (at 175.26 58.42 90))
+    (property "Value" "R_US" (id 1) (at 175.26 60.96 90))
+    (property "Footprint" "" (id 2) (at 175.514 65.786 90)
       (effects (font (size 1.27 1.27)) hide)
     )
-    (property "Footprint" "" (id 2) (at 137.16 110.49 0)
+    (property "Datasheet" "~" (id 3) (at 175.26 64.77 0)
       (effects (font (size 1.27 1.27)) hide)
     )
-    (property "Datasheet" "~" (id 3) (at 137.16 110.49 0)
-      (effects (font (size 1.27 1.27)) hide)
-    )
