File: Schematics/E-Formula.kicad_sch (KiCad schematic)
At the start: 11 parts, among them M1 Motor

Commit message: REFACTOR
Parts:
- removed D1: LED_RED, symbol Device:LED
- removed D2: LED_GREEN, symbol Device:LED
- removed F?: FUSE_LV, symbol Device:Fuse
- removed J?: TSMP-, symbol Connector:Conn_01x01_Male
- removed JP?: HVD, symbol Device:Jumper
- removed Jw?: TSMP+, symbol Connector:Conn_01x01_Male
- removed LV_BATT1: 12V, symbol Device:Battery_Cell
- removed M1: Motor, symbol Motor:Motor_DC
- removed RELAY_DISCHARGE1: TIMED NC, Relay_THT:Relay_SPST_StandexMeder_MS_Form1AB, symbol Relay:MSxx-1Bxx-75
- removed R_DIS1, R_DIS2: 1k, symbol Device:Heater
- added BRAKE_LIGHT2: BRAKE_LIGHT, symbol Device:LED
- added D6: LED_GREEN, symbol Device:LED
- added D7: LED_RED, symbol Device:LED
- added D8: BZV55C12, Diode_SMD:D_MiniMELF, symbol Diode:BZV55C12
- added F2: FUSE_LV, symbol Device:Fuse
- added LV_BATT2: 12V, symbol Device:Battery_Cell
- added M2: MOTOR, symbol A-FA_PARTS:MOTOR
- added M3: PUMP, symbol A-FA_PARTS:PUMP
- added R2: BRAKE, symbol Device:RTRIM
- added RV2: 9851R5KL2.0 APPS, symbol Device:R_Potentiometer_Trim
- added RV3: BRAKE RPS, symbol Device:R_Potentiometer_Trim
- added U2: DC-DC_Converter, symbol A-FA_PARTS:DC-DC_Converter
Connections:
- net GND: now also BRAKE_LIGHT2.1 (K), D8.2 (A), U2.4 (GND)
- net LV: now also D6.2 (A), D7.2 (A), D8.1 (K), R2.2, U2.3 (OUT)
- new net: F2.2, LV_BATT2.1 (+)
- new net: BRAKE_LIGHT2.2 (A), R2.1
- new net BATT+: F2.1, U2.1 (IN)
- new net GNDPWR: LV_BATT2.2 (-), U2.2 (GND)
- new net MOTOR CONTROLLER/A: M2.
- new net MOTOR CONTROLLER/B: M2.
- new net MOTOR CONTROLLER/C: M2.
- new net MOTOR CONTROLLER/PUMP: M3.
Other:
- removed sheet ENERGY METER
- added sheet CHARGE SHUTDOWN (CHARGE_SHUTDOWN.kicad_sch)
- added sheet PRE-MOTOR (PRE_MOTOR.kicad_sch)
- sheet DASHBOARD ports: added 5V_APPS, 5V_RPS, ACC, BMS_LED, BRAKE, BSPD_LED, CRITICAL_LED, GND, GND_APPS, GND_RPS, HVD_LED, IMD_LED, LV, LV_ACTIVE, SHUTDOWN_RESET, SIG_APPS, SIG_RPS, ＣＡＮ＿Ｈ, ＣＡＮ＿Ｌ; removed none
- sheet HV BATTERY PACK ports: added BMS_CHARGE_BUS, BMS_GND, BMS_LV, CAN_H, CAN_L; removed HV_ACTIVE_LIGHT, LV_ACTIVE_LIGHT
- sheet MOTOR CONTROLLER ports: added A, ACC, B, C, CAN＿H, CAN＿L, PUMP; removed OUT+, OUT-
- sheet SHUTDOWN ports: added AIR-_ACTIVE, BMS_LED, BRAKE, BSPD_LED, CRITICAL_LED, GND_BMS, GND_IMD, GND_INV, GND_MCU, GND_PRE, GND_TSAL, HVD_LED, IMD_LED, LV_ACTIVE_INV, LV_ACTIVE_MCU, LV_ACTIVE_PRE, LV_BMS, LV_IMD, LV_INV, LV_MCU, LV_PRE, LV_TSAL, SHUTDOWN_RESET; removed LV, LV_ACTIVE
- note added: "ACC/BRAKE"
- note added: "BRAKE LIGHTINGS"
- note added: "TVS/Zener VI BSPD CHARGE SHUTDOWN DASHBOARD SHUTDOWN INTERFACES"
- note removed: "DISCHARGE"
- note removed: "SHUTDOWN BSPD CHARGE SHUTDOWN DASHBOARD BRAKE/ACC LIGHT"
- note removed: "TSMP"

Commit message: UPDATE
Parts:
- removed D8: BZV55C12, Diode_SMD:D_MiniMELF, symbol Diode:BZV55C12
- removed RV2: 9851R5KL2.0 APPS, symbol Device:R_Potentiometer_Trim
- removed RV3: BRAKE RPS, symbol Device:R_Potentiometer_Trim
- added J?: TSMP-, symbol Connector:Conn_01x01_Male
- added Jw?: TSMP+, symbol Connector:Conn_01x01_Male
- added M4: FAN, symbol A-FA_PARTS:FAN
- added R?: R_US, symbol Device:R_US
- added RESET?: SW_DPST_x2, symbol Switch:SW_Push
- added RV?: BRAKE RPS, symbol Device:R_Potentiometer_Trim
- added RV?: 9851R5KL2.0 APPS, symbol Device:R_Potentiometer_Trim
Connections:
- net GND: now also M4., RESET?.1
- new net: R?.1, RESET?.2
- new net JUNCTION/RAD_FAN_PWR: M4.
- new net SHUTDOWN_RESET: R?.2
Other:
- sheet PRE-MOTOR renamed JUNCTION
- sheet DASHBOARD ports: added none; removed 5V_APPS, 5V_RPS, ACC, GND_APPS, GND_RPS, SHUTDOWN_RESET, SIG_APPS, SIG_RPS
- sheet HV BATTERY PACK ports: added HALL; removed none
- sheet JUNCTION: file PRE_MOTOR.kicad_sch -> JUNCTION.kicad_sch
- sheet JUNCTION ports: added HV_INDICATOR, LV_INDICATOR, RADIATOR_FAN, RAD_FAN_PWR, TSMP+, TSMP-; removed HALL, HV_ACTIVE_LIGHT, LV_ACTIVE_LIGHT
- sheet MOTOR CONTROLLER ports: added BRAKE, RADIATOR_FAN, RESOLVER, TEMP_SENSOR; removed none
- sheet SHUTDOWN ports: added GND_JNC, HALL, LV_ACTIVE_JNC, LV_JNC; removed GND_PRE, GND_TSAL, LV_ACTIVE_PRE, LV_PRE
- note added: "SHUTDOWN RESET BUTTON"
- note added: "TSMP"
- note added: "VI BSPD BSPD SENSOR DASHBOARD CHARGE SHUTDOWN MOTOR CONTROLLER - APPS/BRAKE"
- note removed: "TVS/Zener VI BSPD CHARGE SHUTDOWN DASHBOARD SHUTDOWN INTERFACES"
