File: Schematics/HV_BATTERY_PACK.kicad_sch (KiCad schematic)
At the start: 6 parts

Commit message: REFACTOR
Parts:
- removed FUSE_TRACTIVE: L50QS250.V, symbol Device:Fuse
- removed HV_BATT1: 300V, symbol Device:Battery
- removed RELAY_PRECHARGE1: V23700-C0001-A408, Relay_THT:Relay_StandexMeder_DIP_LowProfile, symbol Relay:DIPxx-1Axx-12x
- removed R_PRE: 1k, symbol Device:Heater
- added CB2: HVD, symbol Device:CircuitBreaker_2P
- added D10, D9: 1N4001, Diode_THT:D_DO-41_SOD81_P10.16mm_Horizontal, symbol Diode:1N4001
- added FUSE_TRACTIVE2: L50QS250.V, symbol Device:Fuse
- added HV_BATT2: 300V, symbol Device:Battery
- added M4: BATT_FAN, symbol Motor:Fan
- added R4: R_PRECHARGE, symbol Device:Heater
- added U3: OrionBMS2-72, symbol A-FA_PARTS:OrionBMS2-72
- added U4: IR155-3204, symbol A-FA_PARTS:IR155-3204
- AIR+2: renamed from AIR+; value LEV200A4ANA -> AIR+
- AIR-2: renamed from AIR-; value LEV200A4ANA -> AIR-
Connections:
- net AIR+_ACTIVE: now also D9.1 (K)
- net AIR-_ACTIVE: now also D10.1 (K)
- net BMS_FAULT: now also U3.7 (DISCHARGE_ENABLE)
- net GND: now also D10.2 (A), D9.2 (A), U4.1 (KI.31), U4.3 (KI.31), U4.4 (KI.31)
- net HV+: now also CB2.1; no longer AIR+2.7, AIR+2.8
- net HV-: now also CB2.3; no longer AIR-2.7, AIR-2.8
- net RELAY_PRECHARGE: now reaches AIR+2.1, AIR+2.14
- net RELAY_PRECHARGE: now also HV_BATT2.1 (+)
- net BMS/BMS-: no longer names the net of AIR-2.1, AIR-2.14
- net BMS/BMS-: now also FUSE_TRACTIVE2.2
- new net: FUSE_TRACTIVE2.1, HV_BATT2.2 (-)
- new net BMS_GND: U3.12 (GND)
- new net BMS_LV: U3.2 (READY_POWER)
- new net CAN_H: U3.18 (CAN1_H)
- new net CAN_L: U3.19 (CAN1_L)
- new net FAN+: M4.1 (+)
- new net FAN-: M4.2 (-)
- new net FAN_ENABLE: U3.10 (FAN_ENABLE)
- new net HV_IMD+: U4.1 (KI.31)
- new net HV_IMD-: U4.1 (KI.31)
- new net HV_SENSE+: AIR+2.7, AIR+2.8, CB2.2, R4.2
- new net HV_SENSE-: AIR-2.7, AIR-2.8, CB2.4
- new net OK_HS: U4.8 (OK_HS)
- new net R_PRECHARGE: R4.1
- new net Vs: U4.2 (KI.15)
- no-connect marks 1 -> 4
Other:
- removed sheet BMS
- removed sheet IMD
- removed sheet TSAL & VOLTAGE INDICATOR
- added sheet BATT_PCB (BATT_PCB.kicad_sch)
- note added: "INTERFACE - CHARGE"
- note added: "INTERFACE - DASHBOARD"
- note added: "INTERFACE - INVERTER"
- note added: "INTERFACE - SHUTDOWN"

Commit message: UPDATE
Other:
- sheet BATT_PCB ports: added HALL; removed none
Changed lines of the file:
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@@
     (stroke (width 0.2) (type default) (color 0 0 0 0))
+  )
+  (wire (pts (xy 208.28 152.4) (xy 210.82 152.4))
+    (stroke (width 0) (type default) (color 0 0 0 0))
   )
   (wire (pts (xy 78.74 93.98) (xy 80.01 93.98))
@@
     (effects (font (size 1.27 1.27) (thickness 0.254) bold) (justify left bottom))
   )
-  (text "INTERFACE - CHARGE" (at 213.36 81.28 0)
+  (text "INTERFACE - CHARGE" (at 213.36 82.55 0)
     (effects (font (size 1.27 1.27) (thickness 0.254) bold) (justify left bottom))
   )
-  (text "INTERFACE - DASHBOARD" (at 213.36 69.85 0)
+  (text "INTERFACE - DASHBOARD" (at 213.36 71.12 0)
     (effects (font (size 1.27 1.27) (thickness 0.254) bold) (justify left bottom))
   )
-  (text "INTERFACE - INVERTER" (at 213.36 59.69 0)
+  (text "INTERFACE - INVERTER" (at 213.36 60.96 0)
     (effects (font (size 1.27 1.27) (thickness 0.254) bold) (justify left bottom))
   )
@@
     )
   )
-  (global_label "CAN_L" (shape input) (at 232.41 74.93 180) (fields_autoplaced)
-    (effects (font (size 1.27 1.27)) (justify right))
-    (property "Intersheet References" "${INTERSHEET_REFS}" (id 0) (at 224.3121 74.8506 0)
+  (global_label "CAN_L" (shape input) (at 232.41 76.2 180) (fields_autoplaced)
+    (effects (font (size 1.27 1.27)) (justify right))
+    (property "Intersheet References" "${INTERSHEET_REFS}" (id 0) (at 224.3121 76.1206 0)
       (effects (font (size 1.27 1.27)) (justify right) hide)
     )
@@
     )
   )
-  (global_label "BMS_CHARGE_BUS" (shape input) (at 232.41 83.82 180) (fields_autoplaced)
+  (global_label "BMS_CHARGE_BUS" (shape input) (at 232.41 85.09 180) (fields_autoplaced)
     (effects (font (size 1.27 1.27) (thickness 0.254) bold) (justify right))
-    (property "Intersheet References" "${INTERSHEET_REFS}" (id 0) (at 212.7522 83.693 0)
+    (property "Intersheet References" "${INTERSHEET_REFS}" (id 0) (at 212.7522 84.963 0)
       (effects (font (size 1.27 1.27) (thickness 0.254) bold) (justify right) hide)
     )
@@
     )
   )
-  (global_label "PRECHARGE" (shape output) (at 232.41 62.23 180) (fields_autoplaced)
-    (effects (font (size 1.27 1.27)) (justify right))
-    (property "Intersheet References" "${INTERSHEET_REFS}" (id 0) (at 218.9298 62.1506 0)
+  (global_label "PRECHARGE" (shape output) (at 232.41 63.5 180) (fields_autoplaced)
+    (effects (font (size 1.27 1.27)) (justify right))
+    (property "Intersheet References" "${INTERSHEET_REFS}" (id 0) (at 218.9298 63.4206 0)
       (effects (font (size 1.27 1.27)) (justify right) hide)
     )
@@
     )
   )
+  (global_label "HALL" (shape output) (at 208.28 152.4 180) (fields_autoplaced)
+    (effects (font (size 1.27 1.27)) (justify right))
+    (property "Intersheet References" "${INTERSHEET_REFS}" (id 0) (at 201.3917 152.3206 0)
+      (effects (font (size 1.27 1.27)) (justify right) hide)
+    )
+  )
   (global_label "RELAY_PRECHARGE" (shape input) (at 208.28 133.35 180) (fields_autoplaced)
     (effects (font (size 1.27 1.27)) (justify right))
@@
     )
   )
-  (global_label "CAN_H" (shape input) (at 232.41 72.39 180) (fields_autoplaced)
-    (effects (font (size 1.27 1.27)) (justify right))
-    (property "Intersheet References" "${INTERSHEET_REFS}" (id 0) (at 224.0098 72.3106 0)
+  (global_label "CAN_H" (shape input) (at 232.41 73.66 180) (fields_autoplaced)
+    (effects (font (size 1.27 1.27)) (justify right))
+    (property "Intersheet References" "${INTERSHEET_REFS}" (id 0) (at 224.0098 73.5806 0)
       (effects (font (size 1.27 1.27)) (justify right) hide)
     )
@@
     )
   )
+  (global_label "HALL" (shape input) (at 232.41 53.34 180) (fields_autoplaced)
+    (effects (font (size 1.27 1.27)) (justify right))
+    (property "Intersheet References" "${INTERSHEET_REFS}" (id 0) (at 225.5217 53.2606 0)
+      (effects (font (size 1.27 1.27)) (justify right) hide)
+    )
+  )
   (global_label "HV_IMD-" (shape input) (at 105.41 116.84 180) (fields_autoplaced)
     (effects (font (size 1.27 1.27)) (justify right))
@@
     )
   )
-  (hierarchical_label "CAN_H" (shape output) (at 232.41 72.39 0)
+  (hierarchical_label "CAN_H" (shape output) (at 232.41 73.66 0)
     (effects (font (size 1.27 1.27) (thickness 0.254) bold) (justify left))
   )
@@
     (effects (font (size 1.27 1.27) (thickness 0.254) bold) (justify left))
   )
-  (hierarchical_label "BMS_CHARGE_BUS" (shape output) (at 232.41 83.82 0)
+  (hierarchical_label "BMS_CHARGE_BUS" (shape output) (at 232.41 85.09 0)
     (effects (font (size 1.27 1.27) (thickness 0.254) bold) (justify left))
   )
@@
     (effects (font (size 1.27 1.27) (thickness 0.254) bold) (justify left))
   )
+  (hierarchical_label "HALL" (shape output) (at 232.41 53.34 0)
+    (effects (font (size 1.27 1.27) (thickness 0.254) bold) (justify left))
+  )
   (hierarchical_label "HV+" (shape output) (at 144.78 78.74 0)
     (effects (font (size 1.27 1.27) (thickness 0.254) bold) (justify left))
   )
-  (hierarchical_label "CAN_L" (shape output) (at 232.41 74.93 0)
-    (effects (font (size 1.27 1.27) (thickness 0.254) bold) (justify left))
-  )
-  (hierarchical_label "PRECHARGE" (shape input) (at 232.41 62.23 0)
+  (hierarchical_label "CAN_L" (shape output) (at 232.41 76.2 0)
+    (effects (font (size 1.27 1.27) (thickness 0.254) bold) (justify left))
+  )
+  (hierarchical_label "PRECHARGE" (shape input) (at 232.41 63.5 0)
     (effects (font (size 1.27 1.27) (thickness 0.254) bold) (justify left))
   )
@@
     (pin "8")
   )
-  (sheet (at 210.82 101.6) (size 43.18 49.53) (fields_autoplaced)
+  (sheet (at 210.82 101.6) (size 43.18 53.34) (fields_autoplaced)
     (stroke (width 0.1524) (type solid) (color 0 0 0 0))
     (fill (color 0 0 0 0.0000))
@@
       (effects (font (size 1.27 1.27)) (justify left bottom))
     )
-    (property "Sheet file" "BATT_PCB.kicad_sch" (id 1) (at 210.82 151.7146 0)
+    (property "Sheet file" "BATT_PCB.kicad_sch" (id 1) (at 210.82 155.5246 0)
       (effects (font (size 1.27 1.27)) (justify left top) hide)
     )
@@
       (effects (font (size 1.27 1.27)) (justify left))
     )
+    (pin "HALL" output (at 210.82 152.4 180)
+      (effects (font (size 1.27 1.27)) (justify left))
+    )
