File: Schematics/JUNCTION.kicad_sch (KiCad schematic)
At the start: 8 parts, among them J2 TSMP-, U9 ENERGY_METER

Commit message: UPDATE
Parts:
- removed J2: TSMP-, symbol Connector:Conn_01x01_Male
- removed Jw2: TSMP+, symbol Connector:Conn_01x01_Male
- removed R21, R22: 10k, symbol Device:R_US
- added R? (x2): 10k, symbol Device:R_US
- added RELAY_RADIATOR_FAN1: TIMED NC, Relay_THT:Relay_SPST_StandexMeder_MS_Form1AB, symbol Relay:MSxx-1Bxx-75
Connections:
- net GND: now also RELAY_RADIATOR_FAN1.5
- net HV_IN+: now also R?.2
- net HV_OUT-: now also R?.2
- net LV: now also RELAY_RADIATOR_FAN1.1
- new net RADIATOR_FAN: RELAY_RADIATOR_FAN1.3
- new net RAD_FAN_PWR: RELAY_RADIATOR_FAN1.7
- new net TSMP+: R?.1
- new net TSMP-: R?.1
Other:
- sheet TSAL ports: added HV_INDICATOR, LV_INDICATOR; removed HV_ACTIVE_LIGHT, LV_ACTIVE_LIGHT
- note added: "INTERFACE - INVERTER"
- note added: "INTERFACE - RADIATOR FAN"
- note added: "INTERFACE - TSMP"
- note added: "RADIATOR FAN"
- note removed: "TSMP"
