File: Schematics/MOTOR_CONTROLLER.kicad_sch (KiCad schematic)
At the start: 0 parts

Commit message: REFACTOR
Changed lines of the file:
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@@
+    (effects (font (size 1.27 1.27)) (justify left))
+  )
+  (hierarchical_label "CAN＿L" (shape output) (at 119.38 114.3 0)
+    (effects (font (size 1.27 1.27)) (justify left))
+  )
+  (hierarchical_label "C" (shape output) (at 139.7 97.79 0)
+    (effects (font (size 1.27 1.27)) (justify left))
+  )
+  (hierarchical_label "ACC" (shape output) (at 119.38 119.38 0)
     (effects (font (size 1.27 1.27)) (justify left))
   )
@@
     (effects (font (size 1.27 1.27)) (justify left))
   )
+  (hierarchical_label "PUMP" (shape output) (at 157.48 86.36 0)
+    (effects (font (size 1.27 1.27)) (justify left))
+  )
   (hierarchical_label "HV+" (shape input) (at 119.38 90.17 0)
     (effects (font (size 1.27 1.27)) (justify left))
   )
-  (hierarchical_label "OUT+" (shape output) (at 139.7 90.17 0)
+  (hierarchical_label "A" (shape output) (at 139.7 90.17 0)
     (effects (font (size 1.27 1.27)) (justify left))
   )
@@
     (effects (font (size 1.27 1.27)) (justify left))
   )
-  (hierarchical_label "OUT-" (shape output) (at 139.7 93.98 0)
+  (hierarchical_label "CAN＿H" (shape output) (at 119.38 111.76 0)
+    (effects (font (size 1.27 1.27)) (justify left))
+  )
+  (hierarchical_label "B" (shape output) (at 139.7 93.98 0)
     (effects (font (size 1.27 1.27)) (justify left))
   )
@@
   (symbol (lib_id "power:GND") (at 161.29 109.22 0) (unit 1)
     (in_bom yes) (on_board yes)
-    (property "Reference" "#PWR?" (id 0) (at 161.29 115.57 0)
+    (property "Reference" "#PWR0121" (id 0) (at 161.29 115.57 0)
       (effects (font (size 1.27 1.27)) hide)
     )

Commit message: UPDATE
Changed lines of the file:
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@@
+    (effects (font (size 1.27 1.27)) (justify left))
+  )
+  (hierarchical_label "TEMP_SENSOR" (shape input) (at 157.48 77.47 0)
+    (effects (font (size 1.27 1.27)) (justify left))
+  )
+  (hierarchical_label "BRAKE" (shape output) (at 119.38 121.92 0)
     (effects (font (size 1.27 1.27)) (justify left))
   )
@@
     (effects (font (size 1.27 1.27)) (justify left))
   )
+  (hierarchical_label "RESOLVER" (shape input) (at 157.48 80.01 0)
+    (effects (font (size 1.27 1.27)) (justify left))
+  )
   (hierarchical_label "AIR+_ACTIVE_SIG" (shape output) (at 157.48 93.98 0)
     (effects (font (size 1.27 1.27)) (justify left))
@@
     (effects (font (size 1.27 1.27)) (justify left))
   )
+  (hierarchical_label "RADIATOR_FAN" (shape output) (at 157.48 83.82 0)
+    (effects (font (size 1.27 1.27)) (justify left))
+  )
