File: Schematics/SHUTDOWN.kicad_sch (KiCad schematic)
At the start: 0 parts

Commit message: REFACTOR
Parts:
- added BOTS1, HV_AUX1, HV_AUX2, HV_AUX3: SW_DPST_x2, symbol Switch:SW_Push_Open
- added D1: BZV55C12, Diode_SMD:D_MiniMELF, symbol Diode:BZV55C12
- added D2, D3, D4, D5: 1N4001, Diode_THT:D_DO-41_SOD81_P10.16mm_Horizontal, symbol Diode:1N4001
- added HV_MASTER1, LV_MASTER1: SW_DPST_x2, symbol Switch:SW_Push
- added JP2: HVD_INTERLOCK, symbol Device:Jumper
- added R1: ?, symbol Device:R_US
- added RELAY_AIR+_ACTIVE2, RELAY_HVD_INTERLOCK1: NOT SPECIFIED, Relay_THT:Relay_StandexMeder_DIP_LowProfile, symbol Relay:DIPxx-1Axx-12x
- added RELAY_BMS2, RELAY_BSPD2, RELAY_IMD2: ADJ14024, symbol NewThing:ADJ14024
Connections:
- net AIR+_ACTIVE: now also RELAY_AIR+_ACTIVE2.1, RELAY_AIR+_ACTIVE2.14
- net AIR+_ACTIVE_SIG: now also RELAY_AIR+_ACTIVE2.13, RELAY_AIR+_ACTIVE2.2
- net BMS_FAULT: now also D3.2 (A), RELAY_BMS2.9 (D)
- net GND: now also D1.2 (A), RELAY_AIR+_ACTIVE2.6, RELAY_HVD_INTERLOCK1.6
- net IMD_FAULT: now also D4.2 (A), RELAY_IMD2.9 (D)
- net LV: now also D2.1 (K), D3.1 (K), D4.1 (K), D5.1 (K), HV_AUX1.1 (A), JP2.1, LV_MASTER1.2, RELAY_BMS2.1 (V), RELAY_BSPD2.1 (V), RELAY_IMD2.1 (V)
- net LV_ACTIVE: now also HV_MASTER1.1, RELAY_AIR+_ACTIVE2.7, RELAY_AIR+_ACTIVE2.8
- net LV_BATT: now also D1.1 (K), LV_MASTER1.1
- new net: BOTS1.1 (A), HV_AUX3.2 (B)
- new net: BOTS1.2 (B), RELAY_HVD_INTERLOCK1.1, RELAY_HVD_INTERLOCK1.14
- new net: HV_MASTER1.2, RELAY_BMS2.4 (12V)
- new net: HV_AUX1.2 (B), HV_AUX2.1 (A)
- new net: RELAY_BSPD2.2 (Out), RELAY_HVD_INTERLOCK1.7, RELAY_HVD_INTERLOCK1.8
- new net: HV_AUX2.2 (B), HV_AUX3.1 (A)
- new net: RELAY_BSPD2.4 (12V), RELAY_IMD2.2 (Out)
- new net: RELAY_BMS2.2 (Out), RELAY_IMD2.4 (12V)
- new net: R1.1, RELAY_BMS2.6 (N), RELAY_BSPD2.6 (N), RELAY_IMD2.6 (N)
- new net BSPD_LED: D5.2 (A), RELAY_BSPD2.9 (D)
- new net CRITICAL_LED: R1.2
- new net HVD_LED: JP2.2, RELAY_HVD_INTERLOCK1.13, RELAY_HVD_INTERLOCK1.2
- new net SHUTDOWN_RESET: D2.2 (A), RELAY_BMS2.8 (L), RELAY_BSPD2.8 (L), RELAY_IMD2.8 (L)
Other:
- added sheet BSPD (BSPD.kicad_sch)
- note added: "20.8mA"
- note added: "HIGH OK LOW FAIL"

Commit message: UPDATE
Parts:
- removed D1: BZV55C12, Diode_SMD:D_MiniMELF, symbol Diode:BZV55C12
- removed D2, D3, D4, D5: 1N4001, Diode_THT:D_DO-41_SOD81_P10.16mm_Horizontal, symbol Diode:1N4001
- removed R1: ?, symbol Device:R_US
- removed RELAY_AIR+_ACTIVE2: NOT SPECIFIED, Relay_THT:Relay_StandexMeder_DIP_LowProfile, symbol Relay:DIPxx-1Axx-12x
- removed RELAY_BMS2, RELAY_BSPD2, RELAY_IMD2: ADJ14024, symbol NewThing:ADJ14024
- added D? (x4): 1N4002, Diode_THT:D_DO-41_SOD81_P10.16mm_Horizontal, symbol Diode:1N4001
- added RELAY_AIR+_ACTIVE?: JQ1-12V-F, Relay_THT:Relay_StandexMeder_DIP_LowProfile, symbol Relay:DIPxx-1Axx-12x
- added RELAY_BMS?, RELAY_BSPD?, RELAY_IMD?: ADJ14012, symbol NewThing:ADJ14024
- added U?: AMS1117-5.0, Package_TO_SOT_SMD:SOT-223-3_TabPin2, symbol Regulator_Linear:AMS1117-5.0
- RELAY_HVD_INTERLOCK1: value NOT SPECIFIED -> JQ1-12V-F
Connections:
- net LV_ACTIVE is gone; now on net AIR-_ACTIVE: HV_MASTER1.1
- net AIR+_ACTIVE: now also RELAY_AIR+_ACTIVE?.1, RELAY_AIR+_ACTIVE?.14
- net AIR+_ACTIVE_SIG: now also RELAY_AIR+_ACTIVE?.13, RELAY_AIR+_ACTIVE?.2
- net AIR-_ACTIVE: now also RELAY_AIR+_ACTIVE?.7, RELAY_AIR+_ACTIVE?.8
- net BMS_FAULT: now also D?.2 (A), RELAY_BMS?.9 (D)
- net CRITICAL_LED: now also RELAY_BMS?.6 (N), RELAY_BSPD?.6 (N), RELAY_IMD?.6 (N)
- net GND: now also RELAY_AIR+_ACTIVE?.6, U?.1 (GND)
- net IMD_FAULT: now also D?.2 (A), RELAY_IMD?.9 (D)
- net LV: now also D?.1 (K), D?.1 (K), D?.1 (K), D?.1 (K), RELAY_BMS?.1 (V), RELAY_BSPD?.1 (V), RELAY_IMD?.1 (V), U?.3 (VI)
- net SHUTDOWN_RESET: now also D?.2 (A), RELAY_BMS?.8 (L), RELAY_BSPD?.8 (L), RELAY_IMD?.8 (L)
- net at HV_MASTER1.2: now also RELAY_BMS?.2 (Out)
- net at RELAY_HVD_INTERLOCK1.7, RELAY_HVD_INTERLOCK1.8: now also RELAY_BSPD?.4 (12V)
- new net: RELAY_BMS?.4 (12V), RELAY_IMD?.2 (Out)
- new net: RELAY_BSPD?.2 (Out), RELAY_IMD?.4 (12V)
- new net 5V: U?.2 (VO)
- new net BSPD_FAULT: D?.2 (A), RELAY_BSPD?.9 (D)
Other:
- sheet BSPD ports: added none; removed BRAKE, BSPD_FAULT, GND, LV
- note added: "INTERFACE - BATTERY PACK"
- note added: "INTERFACE - INVERTER"
- note added: "INTERFACE - JUNCTION"
- note added: "INTERFACE - LV BATT"
- note added: "INTERFACE - MCU"
- note added: "INTERFACE - TSAL"
- note removed: "20.8mA"
- moved on the sheet: BOTS1, HV_AUX1, HV_AUX2, HV_AUX3, HV_MASTER1, LV_MASTER1, RELAY_HVD_INTERLOCK1
