File: Schematics/TSAL.kicad_sch (KiCad schematic)
At the start: 29 parts, among them Q1 IRF640, Q2 IRF640, Q3 IRF640, U1 LM311, U2 4N35, U3 LR8K4-G

Commit message: REFACTOR
Parts:
- removed C3: 2.2uF, symbol Device:C_Small
- removed D2: 1N4758A, Diode_THT:D_DO-41_SOD81_P10.16mm_Horizontal, symbol Diode:1N47xxA
- removed D3: LED, symbol Device:LED
- removed R1, R2, R4: 4.7M, symbol Device:R_US
- removed R14: 18k, symbol Device:R_US
- removed R15: 6k, symbol Device:R_US
- removed R_Sense: 1k, symbol Device:R_US
- removed U3: LR8K4-G, Package_TO_SOT_SMD:TO-252-2, symbol Regulator_Linear:LR8K4-G
- added D12: BZV55C12, Diode_SMD:D_MiniMELF, symbol Diode:BZV55C12
- added R5, R6, R7: 4.7M, symbol Device:R_US
- renumbered C1 to C2, C2 to C3, D1 to D11, PS1 to PS2, Q1 to Q2, Q2 to Q3, Q3 to Q4, R6 to R10, R7 to R11, R8 to R12, R9 to R13, R10 to R14, R11 to R15, R12 to R16, R13 to R17, R5 to R9, U1 to U5, U2 to U6
Connections:
- net GND: now also R16.1, D12.2 (A); no longer R16.2
- net HV+: now also R3.1
- net LV: now also D12.1 (K); no longer Q3.1 (G), Q4.1 (G)
- net at U6.4: now also Q3.1 (G), Q4.1 (G), R16.2; no longer R16.1
- net at C2.2, D11.1 (K), R9.1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: now also R7.2
- net at R3.2: now also R5.1
- new net: R6.2, R7.1
- new net: R5.2, R6.1
Other:
- note added: "A-FA[Ajou University]"
- note removed: "VOLTAGE INDICATOR"
- moved on the sheet: C2, C3, D11, PS2, Q2, Q3, Q4, R10, R11, R12, R13, R14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

Commit message: UPDATE
Parts:
- R14: value 4.7M -> 10k
Connections:
- net HV_ACTIVE_LIGHT renamed HV_INDICATOR
- net LV_ACTIVE_LIGHT renamed LV_INDICATOR
Other:
- moved on the sheet: R3, R5, R6, R7
